Commit message: updated mesh paths

File: kr_description/urdf/kr1018.urdf.xacro (robot description, xacro)
@@ -46,12 +46,12 @@
       <origin rpy="0 0 0" xyz="0 0 0"/>
       <geometry>
-        <mesh filename="package://bunker_description/meshes/kr1018/visual/link_0.stl"/>
-      </geometry>
-      <material name="Grey"/>
-    </visual>
-    <collision>
-      <origin rpy="0 0 0" xyz="0 0 0"/>
-      <geometry>
-        <mesh filename="package://bunker_description/meshes/kr1018/collision/link_0.stl"/>
+        <mesh filename="package://kr_description/meshes/kr1018/visual/link_0.stl"/>
+      </geometry>
+      <material name="Grey"/>
+    </visual>
+    <collision>
+      <origin rpy="0 0 0" xyz="0 0 0"/>
+      <geometry>
+        <mesh filename="package://kr_description/meshes/kr1018/collision/link_0.stl"/>
       </geometry>
       <material name="Grey"/>
@@ -82,12 +82,12 @@
       <origin rpy="0 0 0" xyz="0 0 0"/>
       <geometry>
-        <mesh filename="package://bunker_description/meshes/kr1018/visual/link_1.stl"/>
-      </geometry>
-      <material name="Grey"/>
-    </visual>
-    <collision>
-      <origin rpy="0 0 0" xyz="0 0 0"/>
-      <geometry>
-        <mesh filename="package://bunker_description/meshes/kr1018/collision/link_1.stl"/>
+        <mesh filename="package://kr_description/meshes/kr1018/visual/link_1.stl"/>
+      </geometry>
+      <material name="Grey"/>
+    </visual>
+    <collision>
+      <origin rpy="0 0 0" xyz="0 0 0"/>
+      <geometry>
+        <mesh filename="package://kr_description/meshes/kr1018/collision/link_1.stl"/>
       </geometry>
       <material name="Grey"/>
@@ -112,12 +112,12 @@
       <origin rpy="0 0 0" xyz="0 0 0"/>
       <geometry>
-        <mesh filename="package://bunker_description/meshes/kr1018/visual/link_2.stl"/>
-      </geometry>
-      <material name="Grey"/>
-    </visual>
-    <collision>
-      <origin rpy="0 0 0" xyz="0 0 0"/>
-      <geometry>
-        <mesh filename="package://bunker_description/meshes/kr1018/collision/link_2.stl"/>
+        <mesh filename="package://kr_description/meshes/kr1018/visual/link_2.stl"/>
+      </geometry>
+      <material name="Grey"/>
+    </visual>
+    <collision>
+      <origin rpy="0 0 0" xyz="0 0 0"/>
+      <geometry>
+        <mesh filename="package://kr_description/meshes/kr1018/collision/link_2.stl"/>
       </geometry>
       <material name="Grey"/>
@@ -142,12 +142,12 @@
       <origin rpy="0 0 0" xyz="0 0 0"/>
       <geometry>
-        <mesh filename="package://bunker_description/meshes/kr1018/visual/link_3.stl"/>
-      </geometry>
-      <material name="Grey"/>
-    </visual>
-    <collision>
-      <origin rpy="0 0 0" xyz="0 0 0"/>
-      <geometry>
-        <mesh filename="package://bunker_description/meshes/kr1018/collision/link_3.stl"/>
+        <mesh filename="package://kr_description/meshes/kr1018/visual/link_3.stl"/>
+      </geometry>
+      <material name="Grey"/>
+    </visual>
+    <collision>
+      <origin rpy="0 0 0" xyz="0 0 0"/>
+      <geometry>
+        <mesh filename="package://kr_description/meshes/kr1018/collision/link_3.stl"/>
       </geometry>
       <material name="Grey"/>
@@ -172,12 +172,12 @@
       <origin rpy="0 0 0" xyz="0 0 0"/>
       <geometry>
-        <mesh filename="package://bunker_description/meshes/kr1018/visual/link_4.stl"/>
-      </geometry>
-      <material name="Grey"/>
-    </visual>
-    <collision>
-      <origin rpy="0 0 0" xyz="0 0 0"/>
-      <geometry>
-        <mesh filename="package://bunker_description/meshes/kr1018/collision/link_4.stl"/>
+        <mesh filename="package://kr_description/meshes/kr1018/visual/link_4.stl"/>
+      </geometry>
+      <material name="Grey"/>
+    </visual>
+    <collision>
+      <origin rpy="0 0 0" xyz="0 0 0"/>
+      <geometry>
+        <mesh filename="package://kr_description/meshes/kr1018/collision/link_4.stl"/>
       </geometry>
       <material name="Grey"/>
@@ -202,12 +202,12 @@
       <origin rpy="0 0 0" xyz="0 0 0"/>
       <geometry>
-        <mesh filename="package://bunker_description/meshes/kr1018/visual/link_5.stl"/>
-      </geometry>
-      <material name="Grey"/>
-    </visual>
-    <collision>
-      <origin rpy="0 0 0" xyz="0 0 0"/>
-      <geometry>
-        <mesh filename="package://bunker_description/meshes/kr1018/collision/link_5.stl"/>
+        <mesh filename="package://kr_description/meshes/kr1018/visual/link_5.stl"/>
+      </geometry>
+      <material name="Grey"/>
+    </visual>
+    <collision>
+      <origin rpy="0 0 0" xyz="0 0 0"/>
+      <geometry>
+        <mesh filename="package://kr_description/meshes/kr1018/collision/link_5.stl"/>
       </geometry>
       <material name="Grey"/>
@@ -232,12 +232,12 @@
       <origin rpy="0 0 0" xyz="0 0 0"/>
       <geometry>
-        <mesh filename="package://bunker_description/meshes/kr1018/visual/link_6.stl"/>
-      </geometry>
-      <material name="Grey"/>
-    </visual>
-    <collision>
-      <origin rpy="0 0 0" xyz="0 0 0"/>
-      <geometry>
-        <mesh filename="package://bunker_description/meshes/kr1018/collision/link_6.stl"/>
+        <mesh filename="package://kr_description/meshes/kr1018/visual/link_6.stl"/>
+      </geometry>
+      <material name="Grey"/>
+    </visual>
+    <collision>
+      <origin rpy="0 0 0" xyz="0 0 0"/>
+      <geometry>
+        <mesh filename="package://kr_description/meshes/kr1018/collision/link_6.stl"/>
       </geometry>
       <material name="Grey"/>
@@ -262,12 +262,12 @@
       <origin rpy="0 0 0" xyz="0 0 0"/>
       <geometry>
-        <mesh filename="package://bunker_description/meshes/kr1018/visual/link_7.stl"/>
-      </geometry>
-      <material name="Grey"/>
-    </visual>
-    <collision>
-      <origin rpy="0 0 0" xyz="0 0 0"/>
-      <geometry>
-        <mesh filename="package://bunker_description/meshes/kr1018/collision/link_7.stl"/>
+        <mesh filename="package://kr_description/meshes/kr1018/visual/link_7.stl"/>
+      </geometry>
+      <material name="Grey"/>
+    </visual>
+    <collision>
+      <origin rpy="0 0 0" xyz="0 0 0"/>
+      <geometry>
+        <mesh filename="package://kr_description/meshes/kr1018/collision/link_7.stl"/>
       </geometry>
       <material name="Grey"/>
